Commit message: Plan.md changes

File: jethexa_sim/urdf/jethexa.urdf.xacro (robot description, xacro)
@@ -2,4 +2,5 @@
 <!--
   JetHexa (Hiwonder, Advanced Kit) - simplified simulation model.
+  Targets ROS 2 Humble + Gazebo Harmonic (gz-sim 8).
   18 DoF: 6 legs x (coxa yaw, femur pitch, tibia pitch).
   Link lengths / masses below are PLACEHOLDERS derived from the published
@@ -44,7 +45,4 @@
     <xacro:box_inertial m="${body_mass}" x="${body_x}" y="${body_y}" z="${body_z}"/>
   </link>
-  <gazebo reference="base_link">
-    <material>Gazebo/DarkGrey</material>
-  </gazebo>
   <!-- leg name, mount x, mount y, mount yaw -->
   <xacro:leg name="lf" x="${mount_x}"  y="${mount_y}"  yaw="${radians(45)}"/>
@@ -58,5 +56,5 @@
   <ros2_control name="JetHexaSystem" type="system">
     <hardware>
-      <plugin>gazebo_ros2_control/GazeboSystem</plugin>
+      <plugin>gz_ros2_control/GazeboSimSystem</plugin>
     </hardware>
     <xacro:leg_ifaces leg="lf"/>
@@ -68,5 +66,6 @@
   </ros2_control>
   <gazebo>
-    <plugin filename="libgazebo_ros2_control.so" name="gazebo_ros2_control">
+    <plugin filename="gz_ros2_control-system"
+            name="gz_ros2_control::GazeboSimROS2ControlPlugin">
       <parameters>$(find jethexa_sim)/config/controllers.yaml</parameters>
     </plugin>

File: jethexa_sim/urdf/leg.xacro (robot description, xacro)
@@ -25,5 +25,5 @@
         <material name="jethexa_leg"><color rgba="0.55 0.55 0.58 1"/></material>
       </visual>
-      <collision>
+      <collision name="${name}_coxa_collision">
         <origin xyz="${coxa_len/2} 0 0" rpy="0 ${pi/2} 0"/>
         <geometry><cylinder radius="${seg_r}" length="${coxa_len}"/></geometry>
@@ -47,5 +47,5 @@
         <material name="jethexa_leg"/>
       </visual>
-      <collision>
+      <collision name="${name}_femur_collision">
         <origin xyz="${femur_len/2} 0 0" rpy="0 ${pi/2} 0"/>
         <geometry><cylinder radius="${seg_r}" length="${femur_len}"/></geometry>
@@ -53,5 +53,5 @@
       <xacro:rod_inertial m="${femur_mass}" l="${femur_len}" r="${seg_r}"/>
     </link>
-    <!-- tibia -->
+    <!-- tibia, with the foot as a second collision on the same link -->
     <joint name="${name}_tibia_joint" type="revolute">
       <parent link="${name}_femur_link"/>
@@ -63,4 +63,12 @@
       <dynamics damping="${joint_damping}" friction="${joint_friction}"/>
     </joint>
+    <!--
+      The foot is a named collision on the tibia rather than its own link on a
+      fixed joint. It was originally moved here to dodge sdformat's collision
+      rename - that did not work, because sdformat prefixes EVERY collision
+      with <link>_fixed_joint_lump__, revolute-jointed links included. It is
+      kept this way regardless: six fewer links and six fewer weld constraints
+      for the solver, for no loss, since nothing needs a foot TF frame.
+    -->
     <link name="${name}_tibia_link">
       <visual>
@@ -69,55 +77,41 @@
         <material name="jethexa_leg"/>
       </visual>
-      <collision>
+      <collision name="${name}_shin_collision">
         <origin xyz="${tibia_len/2} 0 0" rpy="0 ${pi/2} 0"/>
         <geometry><cylinder radius="${seg_r*0.8}" length="${tibia_len}"/></geometry>
       </collision>
-      <xacro:rod_inertial m="${tibia_mass}" l="${tibia_len}" r="${seg_r*0.8}"/>
-    </link>
-    <!-- foot: the only link that should touch the ground -->
-    <joint name="${name}_foot_joint" type="fixed">
-      <parent link="${name}_tibia_link"/>
-      <child  link="${name}_foot_link"/>
-      <origin xyz="${tibia_len} 0 0" rpy="0 0 0"/>
-    </joint>
-    <link name="${name}_foot_link">
+      <!-- foot: the only geometry that should normally touch the ground -->
       <visual>
+        <origin xyz="${tibia_len} 0 0" rpy="0 0 0"/>
         <geometry><sphere radius="${foot_r}"/></geometry>
         <material name="jethexa_foot"><color rgba="0.1 0.1 0.1 1"/></material>
       </visual>
-      <collision>
+      <collision name="${name}_foot_collision">
+        <origin xyz="${tibia_len} 0 0" rpy="0 0 0"/>
         <geometry><sphere radius="${foot_r}"/></geometry>
       </collision>
-      <inertial>
-        <mass value="0.01"/>
-        <inertia ixx="1e-6" iyy="1e-6" izz="1e-6" ixy="0" ixz="0" iyz="0"/>
-      </inertial>
+      <xacro:rod_inertial m="${tibia_mass}" l="${tibia_len}" r="${seg_r*0.8}"/>
     </link>
-    <!-- High friction + contact sensor on the feet; the leg segments are
-         low-friction so that scuffing is penalised rather than exploited. -->
-    <gazebo reference="${name}_foot_link">
-      <mu1>1.2</mu1>
-      <mu2>1.2</mu2>
-      <kp>1e6</kp>
-      <kd>100.0</kd>
-      <maxVel>0.0</maxVel>
-      <minDepth>0.001</minDepth>
-      <material>Gazebo/Black</material>
-      <sensor name="${name}_foot_contact" type="contact">
-        <always_on>true</always_on>
-        <update_rate>100</update_rate>
-        <contact><collision>${name}_foot_link_collision</collision></contact>
-        <plugin name="${name}_foot_contact_plugin" filename="libgazebo_ros_bumper.so">
-          <ros>
-            <namespace>/jethexa</namespace>
-            <remapping>bumper_states:=contacts/${name}_foot</remapping>
-          </ros>
-          <frame_name>${name}_foot_link</frame_name>
-        </plugin>
-      </sensor>
-    </gazebo>
-    <gazebo reference="${name}_coxa_link"><mu1>0.3</mu1><mu2>0.3</mu2><material>Gazebo/Grey</material></gazebo>
-    <gazebo reference="${name}_femur_link"><mu1>0.3</mu1><mu2>0.3</mu2><material>Gazebo/Grey</material></gazebo>
-    <gazebo reference="${name}_tibia_link"><mu1>0.3</mu1><mu2>0.3</mu2><material>Gazebo/Grey</material></gazebo>
+    <!--
+      NO FOOT CONTACT SENSORS. Two reasons, in order of importance:
+      1. The real JetHexa has no foot switches, so a policy that consumes foot
+         contact cannot be deployed. The observation space excludes it by
+         design - see docs/jethexa_hardware.md.
+      2. They did not work anyway. Contact sensors on a URDF-spawned model in
+         ROS 2 Humble + Gazebo Harmonic advertise their topic and then publish
+         nothing, whichever collision name they reference. Verified on both the
+         as-written and the sdformat-emitted name.
+      If contact-based reward shaping is wanted later, do it in the MuJoCo
+      training sim, where contacts are directly available - that is where
+      training happens anyway. If Gazebo contacts are genuinely needed, the
+      model has to be authored in SDF rather than converted from URDF.
+      Friction is not set per link at all. <mu1>/<mu2> attach by collision name
+      and sdformat renames collisions, so they silently did nothing and were
+      removed. Contact friction comes from the ground surface in the world file
+      combined with gz's default, which lands near rubber-on-concrete. The cost:
+      we cannot make the feet grippier than the shins, so a policy that learns
+      to shuffle on its shins is not being penalised for it. Fixing that
+      properly means authoring the model in SDF instead of URDF.
+    -->
   </xacro:macro>
 </robot>

File: jethexa_sim/urdf/props.xacro (robot description, xacro)
@@ -19,9 +19,14 @@
   <!-- Spawn height: body clearance when legs are in the default stance. -->
   <xacro:property name="stand_height" value="0.120"/>
-  <!-- Serial-bus servo envelope. Check against the datasheet of the servos
-       actually fitted (HX-35H class, ~35 kg.cm @ 7.4 V) before tuning RL. -->
-  <xacro:property name="joint_limit"    value="2.09"/>   <!-- rad, +/-120 deg -->
-  <xacro:property name="joint_effort"   value="3.4"/>    <!-- N.m -->
-  <xacro:property name="joint_velocity" value="6.5"/>    <!-- rad/s -->
+  <!-- Hiwonder HX-35H serial bus servo, from the datasheet:
+         range    0-240 deg            -> +/-2.094 rad about centre
+         torque   25 kg.cm running, 35 kg.cm stall @ 11.1 V
+                  -> 2.45 N.m running, 3.43 N.m stall
+         speed    0.18 s / 60 deg @ 11.1 V -> 5.82 rad/s
+       We use the RUNNING torque as the limit, not stall: a policy that leans on
+       stall torque is exploiting something the hardware cannot sustain. -->
+  <xacro:property name="joint_limit"    value="2.094"/>  <!-- rad, +/-120 deg -->
+  <xacro:property name="joint_effort"   value="2.45"/>   <!-- N.m, running -->
+  <xacro:property name="joint_velocity" value="5.82"/>   <!-- rad/s, no load -->
   <xacro:property name="joint_damping"  value="0.05"/>
   <xacro:property name="joint_friction" value="0.02"/>

File: jethexa_sim/urdf/sensors.xacro (robot description, xacro)
@@ -2,8 +2,11 @@
 <robot xmlns:xacro="http://www.ros.org/wiki/xacro">
   <!--
-    Sensor payload of the JetHexa Advanced Kit:
+    Sensor payload of the JetHexa Advanced Kit, for Gazebo Harmonic (gz-sim 8):
       - EAI G4 360-deg 2D lidar, mast-mounted above the chassis
       - 3D depth camera (RGB + depth), front-facing
       - IMU on the controller board
+    Sensors publish on gz transport topics. `config/gz_bridge.yaml` maps them
+    onto ROS topics under /jethexa. The world must load the sensors and imu
+    system plugins or these produce nothing - see worlds/flat_ground.sdf.
     Mount poses are approximate; re-measure against the real frame.
   -->
@@ -15,4 +18,10 @@
       <origin xyz="-0.020 0 ${body_z/2 + 0.060}" rpy="0 0 0"/>
     </joint>
+    <!-- Keep this link separate through URDF->SDF conversion, so the sensor
+         sits on its own frame instead of being folded into the chassis. -->
+    <gazebo reference="lidar_joint">
+      <disableFixedJointLumping>true</disableFixedJointLumping>
+      <preserveFixedJoint>true</preserveFixedJoint>
+    </gazebo>
     <link name="lidar_link">
       <visual>
@@ -20,5 +29,5 @@
         <material name="lidar_blue"><color rgba="0.1 0.2 0.5 1"/></material>
       </visual>
-      <collision>
+      <collision name="lidar_collision">
         <geometry><cylinder radius="0.035" length="0.040"/></geometry>
       </collision>
@@ -29,10 +38,11 @@
     </link>
     <gazebo reference="lidar_link">
-      <material>Gazebo/Blue</material>
-      <sensor name="lidar" type="ray">
-        <always_on>true</always_on>
+      <sensor name="lidar" type="gpu_lidar">
+        <topic>scan</topic>
+        <gz_frame_id>lidar_link</gz_frame_id>
+        <always_on>1</always_on>
         <visualize>false</visualize>
-        <update_rate>10.0</update_rate>
-        <ray>
+        <update_rate>10</update_rate>
+        <lidar>
           <scan>
             <horizontal>
@@ -42,4 +52,10 @@
               <max_angle>3.14159</max_angle>
             </horizontal>
+            <vertical>
+              <samples>1</samples>
+              <resolution>1</resolution>
+              <min_angle>0</min_angle>
+              <max_angle>0</max_angle>
+            </vertical>
           </scan>
           <range>
@@ -53,13 +69,5 @@
             <stddev>0.01</stddev>
           </noise>
-        </ray>
-        <plugin name="lidar_plugin" filename="libgazebo_ros_ray_sensor.so">
-          <ros>
-            <namespace>/jethexa</namespace>
-            <remapping>~/out:=scan</remapping>
-          </ros>
-          <output_type>sensor_msgs/LaserScan</output_type>
-          <frame_name>lidar_link</frame_name>
-        </plugin>
+        </lidar>
       </sensor>
     </gazebo>
@@ -70,4 +78,10 @@
       <origin xyz="${body_x/2} 0 0.015" rpy="0 0 0"/>
     </joint>
+    <!-- Keep this link separate through URDF->SDF conversion, so the sensor
+         sits on its own frame instead of being folded into the chassis. -->
+    <gazebo reference="camera_joint">
+      <disableFixedJointLumping>true</disableFixedJointLumping>
+      <preserveFixedJoint>true</preserveFixedJoint>
+    </gazebo>
     <link name="camera_link">
       <visual>
@@ -75,5 +89,5 @@
         <material name="camera_grey"><color rgba="0.2 0.2 0.2 1"/></material>
       </visual>
-      <collision>
+      <collision name="camera_collision">
         <geometry><box size="0.025 0.110 0.030"/></geometry>
       </collision>
@@ -91,8 +105,10 @@
     <link name="camera_optical_frame"/>
     <gazebo reference="camera_link">
-      <material>Gazebo/Grey</material>
-      <sensor name="depth_camera" type="depth">
-        <always_on>true</always_on>
-        <update_rate>15.0</update_rate>
+      <!-- RGB and depth are separate sensors in gz-sim. -->
+      <sensor name="rgb_camera" type="camera">
+        <topic>rgb_camera</topic>
+        <gz_frame_id>camera_optical_frame</gz_frame_id>
+        <always_on>1</always_on>
+        <update_rate>15</update_rate>
         <camera>
           <horizontal_fov>1.047</horizontal_fov>
@@ -103,17 +119,26 @@
           </image>
           <clip>
+            <near>0.05</near>
+            <far>15.0</far>
+          </clip>
+        </camera>
+      </sensor>
+      <sensor name="depth_camera" type="depth_camera">
+        <topic>depth_camera</topic>
+        <gz_frame_id>camera_optical_frame</gz_frame_id>
+        <always_on>1</always_on>
+        <update_rate>15</update_rate>
+        <camera>
+          <horizontal_fov>1.047</horizontal_fov>
+          <image>
+            <width>640</width>
+            <height>480</height>
+            <format>R_FLOAT32</format>
+          </image>
+          <clip>
             <near>0.3</near>
             <far>8.0</far>
           </clip>
         </camera>
-        <plugin name="depth_camera_plugin" filename="libgazebo_ros_camera.so">
-          <ros>
-            <namespace>/jethexa</namespace>
-          </ros>
-          <camera_name>depth_camera</camera_name>
-          <frame_name>camera_optical_frame</frame_name>
-          <min_depth>0.3</min_depth>
-          <max_depth>8.0</max_depth>
-        </plugin>
       </sensor>
     </gazebo>
@@ -124,4 +149,10 @@
       <origin xyz="0 0 ${body_z/2}" rpy="0 0 0"/>
     </joint>
+    <!-- Keep this link separate through URDF->SDF conversion, so the sensor
+         sits on its own frame instead of being folded into the chassis. -->
+    <gazebo reference="imu_joint">
+      <disableFixedJointLumping>true</disableFixedJointLumping>
+      <preserveFixedJoint>true</preserveFixedJoint>
+    </gazebo>
     <link name="imu_link">
       <inertial>
@@ -132,6 +163,8 @@
     <gazebo reference="imu_link">
       <sensor name="imu" type="imu">
-        <always_on>true</always_on>
-        <update_rate>100.0</update_rate>
+        <topic>imu</topic>
+        <gz_frame_id>imu_link</gz_frame_id>
+        <always_on>1</always_on>
+        <update_rate>100</update_rate>
         <imu>
           <angular_velocity>
@@ -146,11 +179,4 @@
           </linear_acceleration>
         </imu>
-        <plugin name="imu_plugin" filename="libgazebo_ros_imu_sensor.so">
-          <ros>
-            <namespace>/jethexa</namespace>
-            <remapping>~/out:=imu</remapping>
-          </ros>
-          <frame_name>imu_link</frame_name>
-        </plugin>
       </sensor>
     </gazebo>
